File: stereo.sch (KiCad schematic (older format))
At the start: 33 parts, among them J1 Phono, J10 Relay Control, J2 Phono, J3 Phono, J4 Phono, J5 Phono, J6 Phono, J7 Phono, J8 Phono, J9 Power In 5V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

Commit message: Added missing pullups on both outputs
Parts:
- added R11, R12: 100K, symbol R
- C9: value 1u -> 100u
Connections:
- net OUT_L: now also R11.2, R12.2
- net at C9.1, R10.1, R3.2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: now also R11.1, R12.1
Changed lines of the file:
@@
 LIBS:valves
 LIBS:particle-boards
+LIBS:stereo-cache
 EELAYER 26 0
 EELAYER END
@@
 Title "Analog Selector"
 Date "2017-04-17"
-Rev "A"
+Rev "B"
 Comp "Thomas Bay"
 Comment1 ""
@@
 P 8950 1900
 F 0 "C9" H 9067 1946 50  0000 L CNN
-F 1 "1u" H 9067 1855 50  0000 L CNN
+F 1 "100u" H 9067 1855 50  0000 L CNN
 F 2 "" H 8988 1750 50  0001 C CNN
 F 3 "" H 8950 1900 50  0001 C CNN
@@
 Connection ~ 7800 1450
 Wire Wire Line
-	7800 2400 7400 2400
+	7400 2400 8950 2400
 Connection ~ 7800 1750
 Wire Wire Line
@@
 Wire Wire Line
 	10150 3400 10250 3400
+$Comp
+L R R11
+U 1 1 591217D0
+P 8650 2700
+F 0 "R11" H 8720 2746 50  0000 L CNN
+F 1 "100K" H 8720 2655 50  0000 L CNN
+F 2 "" V 8580 2700 50  0001 C CNN
+F 3 "" H 8650 2700 50  0001 C CNN
+	1    8650 2700
+	1    0    0    -1
+$EndComp
+$Comp
+L R R12
+U 1 1 5912187E
+P 8950 2700
+F 0 "R12" H 9020 2746 50  0000 L CNN
+F 1 "100K" H 9020 2655 50  0000 L CNN
+F 2 "" V 8880 2700 50  0001 C CNN
+F 3 "" H 8950 2700 50  0001 C CNN
+	1    8950 2700
+	1    0    0    -1
+$EndComp
+Wire Wire Line
+	8650 2400 8650 2550
+Connection ~ 7800 2400
+Wire Wire Line
+	8950 2400 8950 2550
+Connection ~ 8650 2400
+Wire Wire Line
+	8650 2850 8650 4000
+Wire Wire Line
+	8950 2850 8950 4000
+Connection ~ 8950 4000
+Connection ~ 8650 4000
 $EndSCHEMATC

Commit message: Added comment on input level.
Other:
- note added: "SIgnal Levels from BASF preamplifier: +-2,5 V (max)"
Changed lines of the file:
@@
 Connection ~ 8950 4000
 Connection ~ 8650 4000
+Text Notes 850  2950 0    60   ~ 0
+SIgnal Levels from BASF preamplifier: +-2,5 V (max)
 $EndSCHEMATC
